File: kicadFiles/plate/elongatePlate.kicad_pcb (KiCad board)
At the start: 2 copper layers, 300.2 x 91.9 mm, 0 parts

Commit message: Breakout pins, refresh gerbers
Other:
- outline, holes or cut-outs redrawn
Changed lines of the file:
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@@
   (general
     (thickness 1.6)
-    (drawings 410)
+    (drawings 415)
     (tracks 10)
     (zones 0)
@@
     (34 B.Paste user hide)
     (35 F.Paste user hide)
-    (36 B.SilkS user hide)
-    (37 F.SilkS user hide)
+    (36 B.SilkS user)
+    (37 F.SilkS user)
     (38 B.Mask user hide)
     (39 F.Mask user hide)
@@
     (solder_mask_min_width 0.25)
     (aux_axis_origin 9.525 9.525)
-    (grid_origin 9.525 9.525)
     (visible_elements 7FFFFFFF)
     (pcbplotparams
@@
     (uvia_drill 0.1)
   )
+  (gr_arc (start 243.75 138.25) (end 243.75 139.75) (angle -90) (layer F.SilkS) (width 0.15))
+  (gr_arc (start 256 138.25) (end 256 139.75) (angle 90) (layer F.SilkS) (width 0.15))
+  (gr_line (start 246.75 136.75) (end 253 136.75) (layer F.SilkS) (width 0.15))
+  (gr_arc (start 246.75 138.25) (end 246.75 136.75) (angle -90) (layer F.SilkS) (width 0.15))
+  (gr_arc (start 253 138.25) (end 253 136.75) (angle 90) (layer F.SilkS) (width 0.15))
+  (gr_line (start 183.25 136.75) (end 189.5 136.75) (layer F.SilkS) (width 0.15))
+  (gr_arc (start 189.5 138.25) (end 189.5 136.75) (angle 90) (layer F.SilkS) (width 0.15))
+  (gr_arc (start 192.5 138.25) (end 192.5 139.75) (angle 90) (layer F.SilkS) (width 0.15))
+  (gr_arc (start 183.25 138.25) (end 183.25 136.75) (angle -90) (layer F.SilkS) (width 0.15))
+  (gr_arc (start 180.25 138.25) (end 180.25 139.75) (angle -90) (layer F.SilkS) (width 0.15))
+  (gr_arc (start 172.6169 214.4909) (end 166.8669 214.4909) (angle -90) (layer F.SilkS) (width 0.15))
   (gr_line (start 193.789489 220.423382) (end 242.84279 220.423382) (layer Edge.Cuts) (width 0.2))
   (gr_line (start 467.07951 217.883382) (end 467.07951 142.250058) (layer Edge.Cuts) (width 0.2))
@@
   (gr_line (start 443.475561 222.675674) (end 441.967206 221.167311) (layer Edge.Cuts) (width 0.2))
   (gr_curve (pts (xy 441.967206 221.167311) (xy 441.490861 220.690976) (xy 440.844803 220.423377) (xy 440.171156 220.423382)) (layer Edge.Cuts) (width 0.2))
-  (gr_curve (pts (xy 191.993445 138.966108) (xy 192.469785 139.44245) (xy 193.115842 139.710056) (xy 193.789489 139.710058)) (layer Edge.Cuts) (width 0.2))
   (gr_line (start 166.881153 217.883461) (end 166.881153 142.250132) (layer Edge.Cuts) (width 0.2))
-  (gr_curve (pts (xy 188.689037 136.713806) (xy 189.362685 136.713808) (xy 190.008741 136.981414) (xy 190.485082 137.457756)) (layer Edge.Cuts) (width 0.2))
-  (gr_curve (pts (xy 184.443242 136.713806) (xy 184.443242 136.713806) (xy 188.689037 136.713806) (xy 188.689037 136.713806)) (layer Edge.Cuts) (width 0.2))
-  (gr_curve (pts (xy 182.647197 137.457756) (xy 183.123537 136.981414) (xy 183.769594 136.713808) (xy 184.443242 136.713806)) (layer Edge.Cuts) (width 0.2))
-  (gr_curve (pts (xy 181.137961 138.966976) (xy 181.137961 138.966976) (xy 182.647197 137.457756) (xy 182.647197 137.457756)) (layer Edge.Cuts) (width 0.2))
   (gr_curve (pts (xy 252.18904 136.713806) (xy 252.86269 136.713806) (xy 253.50875 136.981412) (xy 253.985092 137.457756)) (layer Edge.Cuts) (width 0.2))
   (gr_curve (pts (xy 247.943244 136.713806) (xy 247.943244 136.713806) (xy 252.18904 136.713806) (xy 252.18904 136.713806)) (layer Edge.Cuts) (width 0.2))
@@
   (gr_line (start 193.789489 139.710058) (end 242.84279 139.710058) (layer Edge.Cuts) (width 0.2))
   (gr_curve (pts (xy 242.84279 139.710058) (xy 243.516439 139.710058) (xy 244.162498 139.442451) (xy 244.638839 138.966108)) (layer Edge.Cuts) (width 0.2))
-  (gr_line (start 190.485082 137.457756) (end 191.993445 138.966108) (layer Edge.Cuts) (width 0.2))
   (gr_line (start 362.367305 158.490903) (end 376.36729 158.490903) (layer Edge.Cuts) (width 0.2))
   (gr_line (start 362.367305 144.490915) (end 362.367305 158.490903) (layer Edge.Cuts) (width 0.2))
@@
   (gr_line (start 300.16729 158.490903) (end 300.16729 144.490915) (layer Edge.Cuts) (width 0.2))
   (gr_curve (pts (xy 329.425 199.925) (xy 330.126401 199.925) (xy 330.695 200.493598) (xy 330.695 201.195)) (layer Edge.Cuts) (width 0.2))
-  (via (at 250.025 138.625) (size 3) (drill 2) (layers F.Cu B.Cu) (net 0))
-  (via (at 186.525 138.625) (size 3) (drill 2) (layers F.Cu B.Cu) (net 0))
+  (via (at 250 138.625) (size 3) (drill 2) (layers F.Cu B.Cu) (net 0))
+  (via (at 186.5 138.625) (size 3) (drill 2) (layers F.Cu B.Cu) (net 0))
   (via (at 383.925 138.625) (size 3) (drill 2) (layers F.Cu B.Cu) (net 0))
   (via (at 316.925 138.625) (size 3) (drill 2) (layers F.Cu B.Cu) (net 0))
