File: kicadFiles/elongate.kicad_pcb (KiCad board)
At the start: 2 copper layers, 294 x 82 mm, 186 parts, among them J1 USB_B_Mini, J3 Conn_01x06_Female, SW1 MXSwitch, SW10 MXSwitch, SW11 MXSwitch, SW12 MXSwitch, SW13 MXSwitch, SW14 MXSwitch, SW15 MXSwitch, SW16 MXSwitch, SW17 MXSwitch, SW18 MXSwitch, SW19 MXSwitch, SW2 MXSwitch, SW20 MXSwitch, SW21 MXSwitch, SW22 MXSwitch, SW23 MXSwitch, SW24 MXSwitch, SW25 MXSwitch, SW26 MXSwitch, SW27 MXSwitch, SW28 MXSwitch, SW29 MXSwitch, SW3 MXSwitch, SW30 MXSwitch, SW31 MXSwitch, SW32 MXSwitch, SW33 MXSwitch, SW34 MXSwitch, SW35 MXSwitch, SW36 MXSwitch, SW37 MXSwitch, SW38 MXSwitch, SW39 MXSwitch, SW4 MXSwitch, SW40 MXSwitch, SW41 MXSwitch, SW42 MXSwitch, SW43 MXSwitch, SW44 MXSwitch, SW45 MXSwitch, SW46 MXSwitch, SW47 MXSwitch, SW48 MXSwitch, SW49 MXSwitch, SW5 MXSwitch, SW50 MXSwitch, SW51 MXSwitch, SW52 MXSwitch, SW53 MXSwitch, SW54 MXSwitch, SW6 MXSwitch, SW7 MXSwitch, SW8 MXSwitch, SW9 MXSwitch, U2 USBLC6-2SC6, U3 ATMEGA32U4, X1 16MHz

Commit message: PCB global deletion and USBC connector port
Parts:
- removed CB1, CU1: 1uF, Capacitor_SMD:C_0805_2012Metric_Pad1.15x1.40mm_HandSolder
- removed CB2, CB3, CB4, CB5, CB6, CRST1: 100nF, Capacitor_SMD:C_0805_2012Metric_Pad1.15x1.40mm_HandSolder
- removed CB7, CB8: 1µ, Capacitor_SMD:C_0805_2012Metric_Pad1.15x1.40mm_HandSolder
- removed CF1: 1u, Capacitor_SMD:C_0805_2012Metric_Pad1.15x1.40mm_HandSolder
- removed CRGB1, CRGB10, CRGB2, CRGB3, CRGB4, CRGB5, CRGB6, CRGB7, CRGB8, CRGB9: 10n, Capacitor_SMD:C_0805_2012Metric_Pad1.15x1.40mm_HandSolder
- removed CX1, CX2: 8.2pF, Capacitor_SMD:C_0805_2012Metric_Pad1.15x1.40mm_HandSolder
- removed J3: Conn_01x06_Female, acheron_Connectors:Conn_AVR_ISP_6
- removed L7: MGFL1608F1R0MT-LF, Inductor_SMD:L_0603_1608Metric
- removed RDM1, RDP1: 22, acheron_Components:R_SMD_1206
- removed RF1: 10k, acheron_Components:R_SMD_1206
- removed RGB1, RGB10, RGB2, RGB3, RGB4, RGB5, RGB6, RGB7, RGB8, RGB9: WS2812B, acheron_Components:LED_WS2812B_5.0x5.0mm_P3.2mm
- removed RGND1: 0R010 1%, Resistor_SMD:R_0805_2012Metric_Pad1.15x1.40mm_HandSolder
- removed RHWB1: 1k, Resistor_SMD:R_0805_2012Metric_Pad1.15x1.40mm_HandSolder
- removed RRGB1, RRGB10, RRGB2, RRGB3, RRGB4, RRGB5, RRGB6, RRGB7, RRGB8, RRGB9: 5R, acheron_Components:R_SMD_1206
- removed RRST1: 4.7k, acheron_Components:R_SMD_1206
- removed RRST2: 330R, acheron_Components:R_SMD_1206
- removed SW_RST1: SW_Push, acheron_Hardware:smdPushBtn
- removed U2: USBLC6-2SC6, acheron_Components:SOT-23-6
- removed U3: ATMEGA32U4, acheron_Components:TQPF-44_10x10mm_P0.8mm
- removed X1: 16MHz, acheron_Components:Crystal_SMD_5032-4Pin_5.0x3.2mm
- added C2: 100n, Capacitor_SMD:C_0805_2012Metric_Pad1.15x1.40mm_HandSolder, F.Cu at (207.4, 153.3)
- added C3: 1u, Capacitor_SMD:C_0805_2012Metric_Pad1.15x1.40mm_HandSolder, F.Cu at (197.9, 166.6)
- added R11: 1M, acheron_Components:R_SMD_1206, F.Cu at (200.2, 166.0)
- added R2: 5.1k, Resistor_SMD:R_0805_2012Metric_Pad1.15x1.40mm_HandSolder, F.Cu at (201.1, 158.0)
- added R3: 5.1k, Resistor_SMD:R_0805_2012Metric_Pad1.15x1.40mm_HandSolder, F.Cu at (195.7, 158.1)
- added R4: 1M, acheron_Components:R_SMD_1206, F.Cu at (205.1, 153.9)
- added U1: TPD4E05U06DQAR, acheron_Components:USON-10_2.5x1.0mm_P0.5mm, F.Cu at (198.4, 157.4)
- F1: value 1A PTC -> Polyfuse
- J1: value USB_B_Mini -> TYPE-C-31-M12_13; footprint acheron_Connectors:USB_MiniB_Hirose_UX60-MB-5S8 -> acheron_Connectors:TYPE-C-31-M-12
- R1: renamed from RSH1; footprint Resistor_SMD:R_0805_2012Metric_Pad1.15x1.40mm_HandSolder -> acheron_Components:R_SMD_1206
- moved L3 130.5 mm to (89.2, 122.5)
- moved F1 12.4 mm to (206.3, 165.5), turned to -90 degrees
- moved D55 7.01 mm to (202.9, 166.3)
- moved R5 3.97 mm to (194.6, 162.5), turned to 90 degrees
- moved C1 3.19 mm to (189.3, 153.4)
- moved R1 1.14 mm to (191.6, 154.1)
- moved J1 0.94 mm to (198.4, 155.5)
- renumbered CSH1 to C1, RI6 to R10, RI1 to R5, RI2 to R6, RI3 to R7, RI4 to R8, RI5 to R9
Connections:
- F1 pad 1: 5V -> VBUS
- F1 pad 2: VBUS -> 5V
Routing:
- net 5V: track 743.1 -> 17.4 mm, vias 7 -> 0
- net Col2: track 629.6 -> 0.00 mm
- net Col3: track 583.3 -> 0.00 mm
- net Col5: track 460.5 -> 0.00 mm
- net Row4: track 346.0 -> 0.00 mm
- net Col10: track 340.7 -> 0.00 mm
- net Row1: track 336.7 -> 0.00 mm
- net Row2: track 324.8 -> 0.00 mm, vias 4 -> 0
- net Col8: track 324.1 -> 0.00 mm
- net Row3: track 316.5 -> 0.00 mm, vias 2 -> 0
- net Col1: track 286.0 -> 0.00 mm
- net Col11: track 273.2 -> 0.00 mm
- net Row5: track 264.4 -> 0.00 mm
- net Col12: track 216.7 -> 0.00 mm
- net Col4: track 212.5 -> 0.00 mm
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- removed copper zone on F.Cu, net GNDD
- removed copper zone on B.Cu, net VDD
Other:
- board size 294 x 82 mm -> 294 x 84.5 mm

Commit message: Change RCC resistors to R0402
Parts:
- removed L3: ElongateLabel, elongateGraphics:elongateLabel
- R2, R3: footprint Resistor_SMD:R_0805_2012Metric_Pad1.15x1.40mm_HandSolder -> Resistor_SMD:R_0402_1005Metric
- moved R3 0.56 mm to (195.7, 157.5)
- moved R2 0.52 mm to (201.0, 157.5)

Commit message: Added LEDs
Parts:
- added LED10: LED, acheron_Components:LED_THT_2.54mm, F.Cu at (212.7, 165.1)
- added LED11: LED, acheron_Components:LED_THT_2.54mm, F.Cu at (231.8, 165.1)
- added LED12: LED, acheron_Components:LED_THT_2.54mm, F.Cu at (250.8, 165.1)
- added LED13: LED, acheron_Components:LED_THT_2.54mm, F.Cu at (269.9, 165.1)
- added LED14: LED, acheron_Components:LED_THT_2.54mm, F.Cu at (288.9, 165.1)
- added LED15: LED, acheron_Components:LED_THT_2.54mm, F.Cu at (308.0, 165.1)
- added LED16: LED, acheron_Components:LED_THT_2.54mm, F.Cu at (327.0, 165.1)
- added LED17: LED, acheron_Components:LED_THT_2.54mm, F.Cu at (346.1, 165.1)
- added LED18: LED, acheron_Components:LED_THT_2.54mm, F.Cu at (365.1, 165.1)
- added LED19: LED, acheron_Components:LED_THT_2.54mm, F.Cu at (384.2, 165.1)
- added LED20: LED, acheron_Components:LED_THT_2.54mm, F.Cu at (403.2, 165.1)
- added LED21: LED, acheron_Components:LED_THT_2.54mm, F.Cu at (422.3, 165.1)
- added LED22: LED, acheron_Components:LED_THT_2.54mm, F.Cu at (146.0, 184.1)
- added LED23: LED, acheron_Components:LED_THT_2.54mm, F.Cu at (165.1, 184.1)
- added LED24: LED, acheron_Components:LED_THT_2.54mm, F.Cu at (184.1, 184.1)
- added LED25: LED, acheron_Components:LED_THT_2.54mm, F.Cu at (219.8, 184.1)
- added LED26: LED, acheron_Components:LED_THT_2.54mm, F.Cu at (246.0, 184.1)
- added LED27: LED, acheron_Components:LED_THT_2.54mm, F.Cu at (265.1, 184.1)
- added LED28: LED, acheron_Components:LED_THT_2.54mm, F.Cu at (284.1, 184.1)
- added LED29: LED, acheron_Components:LED_THT_2.54mm, F.Cu at (303.2, 184.1)
- added LED30: LED, acheron_Components:LED_THT_2.54mm, F.Cu at (322.2, 184.1)
- added LED31: LED, acheron_Components:LED_THT_2.54mm, F.Cu at (341.3, 184.1)
- added LED32: LED, acheron_Components:LED_THT_2.54mm, F.Cu at (360.3, 184.1)
- added LED33: LED, acheron_Components:LED_THT_2.54mm, F.Cu at (379.4, 184.1)
- added LED34: LED, acheron_Components:LED_THT_2.54mm, F.Cu at (398.4, 184.1)
- added LED35: LED, acheron_Components:LED_THT_2.54mm, F.Cu at (419.9, 184.1)
- added LED36: LED, acheron_Components:LED_THT_2.54mm, F.Cu at (146.0, 203.2)
- added LED37: LED, acheron_Components:LED_THT_2.54mm, F.Cu at (165.1, 203.2)
- added LED38: LED, acheron_Components:LED_THT_2.54mm, F.Cu at (184.1, 203.2)
- added LED39: LED, acheron_Components:LED_THT_2.54mm, F.Cu at (207.9, 207.9)
- added LED40: LED, acheron_Components:LED_THT_2.54mm, F.Cu at (234.1, 203.2)
- added LED41: LED, acheron_Components:LED_THT_2.54mm, F.Cu at (255.6, 203.2)
- added LED42: LED, acheron_Components:LED_THT_2.54mm, F.Cu at (274.6, 203.2)
- added LED43: LED, acheron_Components:LED_THT_2.54mm, F.Cu at (293.7, 203.2)
- added LED44: LED, acheron_Components:LED_THT_2.54mm, F.Cu at (312.7, 203.2)
- added LED45: LED, acheron_Components:LED_THT_2.54mm, F.Cu at (331.8, 203.2)
- added LED46: LED, acheron_Components:LED_THT_2.54mm, F.Cu at (350.8, 203.2)
- added LED47: LED, acheron_Components:LED_THT_2.54mm, F.Cu at (369.9, 203.2)
- added LED48: LED, acheron_Components:LED_THT_2.54mm, F.Cu at (388.9, 203.2)
- added LED49: LED, acheron_Components:LED_THT_2.54mm, F.Cu at (415.1, 203.2)
- added LED50: LED, acheron_Components:LED_THT_2.54mm, F.Cu at (146.0, 222.2)
- added LED51: LED, acheron_Components:LED_THT_2.54mm, F.Cu at (165.1, 222.2)
- added LED52: LED, acheron_Components:LED_THT_2.54mm, F.Cu at (188.9, 227.0)
- added LED53: LED, acheron_Components:LED_THT_2.54mm, F.Cu at (207.9, 227.0)
- added LED54: LED, acheron_Components:LED_THT_2.54mm, F.Cu at (227.0, 227.0)
- added LED55: LED, acheron_Components:LED_THT_2.54mm, F.Cu at (250.8, 222.2)
- added LED56: LED, acheron_Components:LED_THT_2.54mm, F.Cu at (286.5, 222.2)
- added LED57: LED, acheron_Components:LED_THT_2.54mm, F.Cu at (343.7, 222.2)
- added LED58: LED, acheron_Components:LED_THT_2.54mm, F.Cu at (377.0, 222.2)
- added LED59: LED, acheron_Components:LED_THT_2.54mm, F.Cu at (398.4, 222.2)
- added LED60: LED, acheron_Components:LED_THT_2.54mm, F.Cu at (419.9, 222.2)
- added LED7: LED, acheron_Components:LED_THT_2.54mm, F.Cu at (146.0, 165.1)
- added LED8: LED, acheron_Components:LED_THT_2.54mm, F.Cu at (165.1, 165.1)
- added LED9: LED, acheron_Components:LED_THT_2.54mm, F.Cu at (184.1, 165.1)
- added Q1: AO3401A, Package_TO_SOT_SMD:SOT-23, F.Cu at (331.4, 284.9)
- added Q2: DTC123JKAT146, Package_TO_SOT_SMD:SOT-23, F.Cu at (326.1, 288.1)
- added R12: 10k, acheron_Components:R_SMD_1206, F.Cu at (315.6, 284.7)
- added R13: 100R, acheron_Components:R_SMD_1206, F.Cu at (309.7, 288.0)
- added R14: 390R, acheron_Components:R_SMD_1206, F.Cu at (309.7, 281.5)
- added R15: 390R, acheron_Components:R_SMD_1206, F.Cu at (315.6, 281.5)
- added R16: 390R, acheron_Components:R_SMD_1206, F.Cu at (309.7, 291.3)
- added R17: 390R, acheron_Components:R_SMD_1206, F.Cu at (321.6, 281.5)
- added R18: 390R, acheron_Components:R_SMD_1206, F.Cu at (309.7, 284.7)
- added R19: 390R, acheron_Components:R_SMD_1206, F.Cu at (315.6, 288.0)
- added R20: 390R, acheron_Components:R_SMD_1206, F.Cu at (370.2, 282.5)
- added R21: 390R, acheron_Components:R_SMD_1206, F.Cu at (370.2, 279.2)
- added R22: 390R, acheron_Components:R_SMD_1206, F.Cu at (364.2, 285.8)
- added R23: 390R, acheron_Components:R_SMD_1206, F.Cu at (364.2, 282.5)
- added R24: 390R, acheron_Components:R_SMD_1206, F.Cu at (364.2, 279.2)
- added R25: 390R, acheron_Components:R_SMD_1206, F.Cu at (428.0, 271.6)
- added R26: 390R, acheron_Components:R_SMD_1206, F.Cu at (433.9, 271.6)
- added R27: 390R, acheron_Components:R_SMD_1206, F.Cu at (428.0, 274.9)
- added R28: 390R, acheron_Components:R_SMD_1206, F.Cu at (428.0, 278.1)
- added R29: 390R, acheron_Components:R_SMD_1206, F.Cu at (355.6, 345.5)
- added R30: 390R, acheron_Components:R_SMD_1206, F.Cu at (373.4, 345.5)
- added R31: 390R, acheron_Components:R_SMD_1206, F.Cu at (367.5, 338.9)
- added R32: 390R, acheron_Components:R_SMD_1206, F.Cu at (349.6, 361.9)
- added R33: 390R, acheron_Components:R_SMD_1206, F.Cu at (349.6, 348.8)
- added R34: 390R, acheron_Components:R_SMD_1206, F.Cu at (361.5, 345.5)
- added R35: 390R, acheron_Components:R_SMD_1206, F.Cu at (373.4, 338.9)
- added R36: 390R, acheron_Components:R_SMD_1206, F.Cu at (349.6, 352.1)
- added R37: 390R, acheron_Components:R_SMD_1206, F.Cu at (373.4, 342.2)
- added R38: 390R, acheron_Components:R_SMD_1206, F.Cu at (349.6, 355.3)
- added R39: 390R, acheron_Components:R_SMD_1206, F.Cu at (379.4, 338.9)
- added R40: 390R, acheron_Components:R_SMD_1206, F.Cu at (349.6, 345.5)
- added R41: 390R, acheron_Components:R_SMD_1206, F.Cu at (361.5, 338.9)
- added R42: 390R, acheron_Components:R_SMD_1206, F.Cu at (361.5, 355.3)
- added R43: 390R, acheron_Components:R_SMD_1206, F.Cu at (355.6, 352.1)
- added R44: 390R, acheron_Components:R_SMD_1206, F.Cu at (361.5, 342.2)
- added R45: 390R, acheron_Components:R_SMD_1206, F.Cu at (355.6, 355.3)
- added R46: 390R, acheron_Components:R_SMD_1206, F.Cu at (355.6, 358.6)
- added R47: 390R, acheron_Components:R_SMD_1206, F.Cu at (349.6, 358.6)
- added R48: 390R, acheron_Components:R_SMD_1206, F.Cu at (355.6, 361.9)
- added R49: 390R, acheron_Components:R_SMD_1206, F.Cu at (355.6, 338.9)
- added R50: 390R, acheron_Components:R_SMD_1206, F.Cu at (367.5, 342.2)
- added R51: 390R, acheron_Components:R_SMD_1206, F.Cu at (355.6, 348.8)
- added R52: 390R, acheron_Components:R_SMD_1206, F.Cu at (367.5, 348.8)
- added R53: 390R, acheron_Components:R_SMD_1206, F.Cu at (349.6, 342.2)
- added R54: 390R, acheron_Components:R_SMD_1206, F.Cu at (361.5, 348.8)
- added R55: 390R, acheron_Components:R_SMD_1206, F.Cu at (361.5, 352.1)
- added R56: 390R, acheron_Components:R_SMD_1206, F.Cu at (355.6, 342.2)
- added R57: 390R, acheron_Components:R_SMD_1206, F.Cu at (461.3, 353.7)
- added R58: 390R, acheron_Components:R_SMD_1206, F.Cu at (455.4, 357.0)
- added R59: 390R, acheron_Components:R_SMD_1206, F.Cu at (455.4, 353.7)
- added R60: 390R, acheron_Components:R_SMD_1206, F.Cu at (473.2, 350.4)
- added R61: 390R, acheron_Components:R_SMD_1206, F.Cu at (455.4, 347.1)
- added R62: 390R, acheron_Components:R_SMD_1206, F.Cu at (473.2, 347.1)
- added R63: 390R, acheron_Components:R_SMD_1206, F.Cu at (461.3, 347.1)
- added R64: 390R, acheron_Components:R_SMD_1206, F.Cu at (461.3, 350.4)
- added R65: 390R, acheron_Components:R_SMD_1206, F.Cu at (455.4, 350.4)
- added R66: 390R, acheron_Components:R_SMD_1206, F.Cu at (467.3, 350.4)
- added R67: 390R, acheron_Components:R_SMD_1206, F.Cu at (461.3, 357.0)
- moved L2 218.1 mm to (170.8, 208.4)
- moved D23 7.04 mm to (236.5, 182.9)
- moved L4 3.36 mm to (398.9, 189.2)
- moved L1 2.83 mm to (294.7, 188.7)
- renumbered C2 to C1, C1 to C2, D16 to D14, D17 to D15, D18 to D16, D19 to D17, D20 to D18, D21 to D19, D22 to D20, D23 to D21, D24 to D22, D25 to D23, D26 to D24, D27 to D25, D30 to D26, D31 to D27, D32 to D28, D33 to D29, D34 to D30, D35 to D31, D36 to D32, D37 to D33, D38 to D34, D39 to D35, D40 to D36, D41 to D37, D44 to D38, D45 to D39, D46 to D40, D47 to D41, D48 to D42, D49 to D43, D50 to D44, D51 to D45, D52 to D46, D42 to D47, D53 to D48, D15 to D49, D29 to D50, D43 to D51, D54 to D52, D14 to D53, D28 to D54, R2 to R1, R3 to R2, R4 to R3, R1 to R4, SW16 to SW14, SW17 to SW15, SW18 to SW16, SW19 to SW17, SW20 to SW18, SW21 to SW19, SW22 to SW20, SW23 to SW21, SW24 to SW22, SW25 to SW23, SW26 to SW24, SW27 to SW25, SW30 to SW26, SW31 to SW27, SW32 to SW28, SW33 to SW29, SW34 to SW30, SW35 to SW31, SW36 to SW32, SW37 to SW33, SW38 to SW34, SW39 to SW35, SW40 to SW36, SW41 to SW37, SW44 to SW38, SW45 to SW39, SW46 to SW40, SW47 to SW41, SW48 to SW42, SW49 to SW43, SW50 to SW44, SW51 to SW45, SW52 to SW46, SW42 to SW47, SW53 to SW48, SW15 to SW49, SW29 to SW50, SW43 to SW51, SW54 to SW52, SW14 to SW53, SW28 to SW54
Routing:
- added copper zone on B.Cu, net (none)

Commit message: Finish LED placin, add MCU
Parts:
- added J2: AVR-JTAG-10, acheron_Connectors:Conn_ARM_JTAG_SWD_10, F.Cu at (263.9, 217.1)
- added U2: STM32F072CBT6, acheron_Components:LQFP-48_7x7mm_P0.5mm, F.Cu at (218.9, 194.8)
- moved R57 340.7 mm to (146.0, 224.6), turned to 180 degrees
- moved R58 319.0 mm to (165.1, 224.6), turned to 180 degrees
- moved R59 294.1 mm to (188.9, 229.4), turned to 180 degrees
- moved R60 291.6 mm to (207.9, 229.4), turned to 180 degrees
- moved R29 263.0 mm to (146.0, 186.5), turned to 180 degrees
- moved R30 262.1 mm to (165.1, 186.5), turned to 180 degrees
- moved R61 256.9 mm to (227.0, 229.4), turned to 180 degrees
- moved R43 255.7 mm to (146.0, 205.5), turned to 180 degrees
- moved R62 253.9 mm to (250.8, 224.6), turned to 180 degrees
- moved R44 239.3 mm to (165.1, 205.5), turned to 180 degrees
- moved R31 238.4 mm to (184.1, 186.5), turned to 180 degrees
- moved R45 227.7 mm to (184.1, 205.5), turned to 180 degrees
- moved R32 223.4 mm to (214.4, 184.1)
- moved R63 213.5 mm to (286.5, 224.6), turned to 180 degrees
- moved R46 209.3 mm to (207.9, 210.3), turned to 180 degrees
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Connections:
- D47 pad 1: Row5 -> Row3
- D48 pad 1: Row5 -> Row4
- D49 pad 1: Row5 -> Row1
- D50 pad 1: Row5 -> Row2
- D51 pad 1: Row5 -> Row3
- D52 pad 1: Row5 -> Row4
- D53 pad 1: Row5 -> Row1
- D54 pad 1: Row5 -> Row2
- SW47 pad 1: Col12 -> Col14
- SW48 pad 1: Col13 -> Col14
- SW49 pad 1: Col2 -> Col15
- SW50 pad 1: Col3 -> Col15
- SW51 pad 1: Col5 -> Col15
- SW52 pad 1: Col8 -> Col15
- SW53 pad 1: Col10 -> Col14
- SW54 pad 1: Col11 -> Col14
Routing:
- net D+: track 20.1 -> 70.7 mm, vias 2 -> 3
- net D-: track 18.2 -> 67.5 mm, vias 2 -> 3
- net Net-(LED4-PadA): track 0.00 -> 3.34 mm
- net Net-(LED5-PadA): track 0.00 -> 3.34 mm
- net Net-(LED6-PadA): track 0.00 -> 3.34 mm
Other:
- board text added: "SWD"

Commit message: Almost finish routing, DRC pending
Parts:
- added C10: 1u, Capacitor_SMD:C_0805_2012Metric_Pad1.15x1.40mm_HandSolder, F.Cu at (191.0, 175.4)
- added C11: 1u, Capacitor_SMD:C_0805_2012Metric_Pad1.15x1.40mm_HandSolder, F.Cu at (148.2, 170.9)
- added C12: 1u, Capacitor_SMD:C_0805_2012Metric_Pad1.15x1.40mm_HandSolder, F.Cu at (152.0, 211.9)
- added C13: 1u, Capacitor_SMD:C_0805_2012Metric_Pad1.15x1.40mm_HandSolder, F.Cu at (197.5, 209.5)
- added C14: 1u, Capacitor_SMD:C_0805_2012Metric_Pad1.15x1.40mm_HandSolder, F.Cu at (229.6, 209.4)
- added C15: 1u, Capacitor_SMD:C_0805_2012Metric_Pad1.15x1.40mm_HandSolder, F.Cu at (267.7, 209.3)
- added C16: 1u, Capacitor_SMD:C_0805_2012Metric_Pad1.15x1.40mm_HandSolder, F.Cu at (312.9, 209.3)
- added C17: 1u, Capacitor_SMD:C_0805_2012Metric_Pad1.15x1.40mm_HandSolder, F.Cu at (346.3, 207.0)
- added C18: 1u, Capacitor_SMD:C_0805_2012Metric_Pad1.15x1.40mm_HandSolder, F.Cu at (383.3, 207.0)
- added C19: 1u, Capacitor_SMD:C_0805_2012Metric_Pad1.15x1.40mm_HandSolder, F.Cu at (420.2, 207.5)
- added C20: 100u, Capacitor_SMD:C_0805_2012Metric_Pad1.15x1.40mm_HandSolder, F.Cu at (278.9, 210.8)
- added C21: 10u, Capacitor_SMD:C_0805_2012Metric_Pad1.15x1.40mm_HandSolder, F.Cu at (262.1, 217.9)
- added C4: 1u, Capacitor_SMD:C_0805_2012Metric_Pad1.15x1.40mm_HandSolder, F.Cu at (405.7, 170.7)
- added C5: 1u, Capacitor_SMD:C_0805_2012Metric_Pad1.15x1.40mm_HandSolder, F.Cu at (367.5, 170.8)
- added C6: 1u, Capacitor_SMD:C_0805_2012Metric_Pad1.15x1.40mm_HandSolder, F.Cu at (329.3, 171.2)
- added C7: 1u, Capacitor_SMD:C_0805_2012Metric_Pad1.15x1.40mm_HandSolder, F.Cu at (291.1, 171.0)
- added C8: 1u, Capacitor_SMD:C_0805_2012Metric_Pad1.15x1.40mm_HandSolder, F.Cu at (253.0, 171.0)
- added C9: 1u, Capacitor_SMD:C_0805_2012Metric_Pad1.15x1.40mm_HandSolder, F.Cu at (214.9, 170.8)
- added D56: WS2812C, acheron_Components:LED_WS2812B_5.0x5.0mm_P3.2mm, F.Cu at (412.8, 169.0)
- added D57: WS2812C, acheron_Components:LED_WS2812B_5.0x5.0mm_P3.2mm, F.Cu at (374.6, 168.6)
- added D58: WS2812C, acheron_Components:LED_WS2812B_5.0x5.0mm_P3.2mm, F.Cu at (336.5, 168.6)
- added D59: WS2812C, acheron_Components:LED_WS2812B_5.0x5.0mm_P3.2mm, F.Cu at (298.4, 168.6)
- added D60: WS2812C, acheron_Components:LED_WS2812B_5.0x5.0mm_P3.2mm, F.Cu at (260.3, 168.3)
- added D61: WS2812C, acheron_Components:LED_WS2812B_5.0x5.0mm_P3.2mm, F.Cu at (222.2, 168.3)
- added D62: WS2812C, acheron_Components:LED_WS2812B_5.0x5.0mm_P3.2mm, F.Cu at (190.1, 168.3)
- added D63: WS2812C, acheron_Components:LED_WS2812B_5.0x5.0mm_P3.2mm, F.Cu at (155.6, 168.3)
- added D64: WS2812C, acheron_Components:LED_WS2812B_5.0x5.0mm_P3.2mm, F.Cu at (155.6, 207.9)
- added D65: WS2812C, acheron_Components:LED_WS2812B_5.0x5.0mm_P3.2mm, F.Cu at (190.1, 210.3)
- added D66: WS2812C, acheron_Components:LED_WS2812B_5.0x5.0mm_P3.2mm, F.Cu at (222.2, 210.3)
- added D67: WS2812C, acheron_Components:LED_WS2812B_5.0x5.0mm_P3.2mm, F.Cu at (260.3, 210.0)
- added D68: WS2812C, acheron_Components:LED_WS2812B_5.0x5.0mm_P3.2mm, F.Cu at (305.6, 210.0)
- added D69: WS2812C, acheron_Components:LED_WS2812B_5.0x5.0mm_P3.2mm, F.Cu at (338.9, 207.6)
- added D70: WS2812C, acheron_Components:LED_WS2812B_5.0x5.0mm_P3.2mm, F.Cu at (375.8, 207.6)
- added D71: WS2812C, acheron_Components:LED_WS2812B_5.0x5.0mm_P3.2mm, F.Cu at (412.7, 207.6)
- added D72: 1N4148, acheron_Components:D_SOD-123, F.Cu at (276.6, 214.6)
- added J3: Conn_01x11, acheron_Connectors:PinHeader_2x5_P2.54mm_Vertical, F.Cu at (212.0, 212.6)
- added Q3: AO3401A, Package_TO_SOT_SMD:SOT-23, F.Cu at (422.8, 173.2)
- added Q4: DTC123JKAT146, Package_TO_SOT_SMD:SOT-23, F.Cu at (262.0, 214.8)
- added R68: 3R, acheron_Components:R_SMD_1206, F.Cu at (408.0, 169.8)
- added R69: 3R, acheron_Components:R_SMD_1206, F.Cu at (369.8, 169.9)
- added R70: 3R, acheron_Components:R_SMD_1206, F.Cu at (331.7, 170.3)
- added R71: 3R, acheron_Components:R_SMD_1206, F.Cu at (293.5, 170.1)
- added R72: 3R, acheron_Components:R_SMD_1206, F.Cu at (255.4, 170.0)
- added R73: 3R, acheron_Components:R_SMD_1206, F.Cu at (217.3, 169.8)
- added R74: 3R, acheron_Components:R_SMD_1206, F.Cu at (193.4, 174.7)
- added R75: 3R, acheron_Components:R_SMD_1206, F.Cu at (150.6, 169.8)
- added R76: 3R, acheron_Components:R_SMD_1206, F.Cu at (156.6, 212.1)
- added R77: 3R, acheron_Components:R_SMD_1206, F.Cu at (194.9, 209.9)
- added R78: 3R, acheron_Components:R_SMD_1206, F.Cu at (227.2, 209.8)
- added R79: 3R, acheron_Components:R_SMD_1206, F.Cu at (265.3, 209.5)
- added R80: 3R, acheron_Components:R_SMD_1206, F.Cu at (310.5, 209.6)
- added R81: 3R, acheron_Components:R_SMD_1206, F.Cu at (343.9, 207.2)
- added R82: 3R, acheron_Components:R_SMD_1206, F.Cu at (380.9, 207.1)
- added R83: 3R, acheron_Components:R_SMD_1206, F.Cu at (417.8, 207.0)
- added R84: 10k, acheron_Components:R_SMD_1206, F.Cu at (422.3, 170.0)
- added R85: 5.1k, acheron_Components:R_SMD_1206, F.Cu at (427.4, 170.0)
- added R86: 10k, acheron_Components:R_SMD_1206, F.Cu at (427.4, 172.6)
- added R87: 100k, acheron_Components:R_SMD_1206, F.Cu at (279.2, 214.7)
- added R88: 100R, acheron_Components:R_SMD_1206, F.Cu at (259.0, 215.5)
- added R89: 33k, acheron_Components:R_SMD_1206, F.Cu at (274.1, 214.7)
- added SW55: SW_Push, acheron_Hardware:smdPushBtn, F.Cu at (268.4, 217.0)
- J2: value AVR-JTAG-10 -> Conn_ARM_JTAG_SWD_10
- moved Q2 128.0 mm to (240.8, 192.7)
- moved Q1 123.3 mm to (249.4, 192.7)
- moved R13 115.7 mm to (243.8, 192.9), turned to 90 degrees
- moved R12 115.0 mm to (246.4, 192.9), turned to 90 degrees
- moved J2 61.5 mm to (325.4, 216.9)
- moved R8 6.66 mm to (317.5, 209.0), turned to 180 degrees
- moved R56 6.54 mm to (421.1, 202.8)
- moved R46 5.50 mm to (203.0, 208.0), turned to 0 degrees
- moved D39 3.57 mm to (244.8, 198.1), turned to 90 degrees
- moved D31 3.57 mm to (398.4, 198.1), turned to 90 degrees
- moved D32 3.57 mm to (379.4, 198.1), turned to 90 degrees
- moved D33 3.57 mm to (360.3, 198.1), turned to 90 degrees
- moved D34 3.57 mm to (341.3, 198.1), turned to 90 degrees
- moved D35 3.57 mm to (322.2, 198.1), turned to 90 degrees
- moved D36 3.57 mm to (303.2, 198.1), turned to 90 degrees
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- renumbered D53 to D14, D49 to D15, D14 to D16, D15 to D17, D16 to D18, D17 to D19, D18 to D20, D19 to D21, D20 to D22, D21 to D23, D22 to D24, D23 to D25, D24 to D26, D25 to D27, D54 to D28, D50 to D29, D26 to D30, D27 to D31, D28 to D32, D29 to D33, D30 to D34, D31 to D35, D32 to D36, D33 to D37, D34 to D38, D35 to D39, D36 to D40, D37 to D41, D47 to D42, D51 to D43, D38 to D44, D39 to D45, D40 to D46, D41 to D47, D42 to D48, D43 to D49, D44 to D50, D45 to D51, D46 to D52, D48 to D53, D52 to D54, SW53 to SW14, SW49 to SW15, SW14 to SW16, SW15 to SW17, SW16 to SW18, SW17 to SW19, SW18 to SW20, SW19 to SW21, SW20 to SW22, SW21 to SW23, SW22 to SW24, SW23 to SW25, SW24 to SW26, SW25 to SW27, SW54 to SW28, SW50 to SW29, SW26 to SW30, SW27 to SW31, SW28 to SW32, SW29 to SW33, SW30 to SW34, SW31 to SW35, SW32 to SW36, SW33 to SW37, SW34 to SW38, SW35 to SW39, SW36 to SW40, SW37 to SW41, SW47 to SW42, SW51 to SW43, SW38 to SW44, SW39 to SW45, SW40 to SW46, SW41 to SW47, SW42 to SW48, SW43 to SW49, SW44 to SW50, SW45 to SW51, SW46 to SW52, SW48 to SW53, SW52 to SW54
Connections:
- J2 pad 10: Net-(J2-Pad10) -> nRST
- J2 pad 2: Net-(J2-Pad10) -> SWDIO
- J2 pad 3: Net-(J2-Pad3) -> GND
- J2 pad 4: Net-(J2-Pad4) -> SWCLK
- J2 pad 5: Net-(J2-Pad5) -> GND
- J2 pad 9: Net-(J2-Pad9) -> GND
- U2 pad 1: Net-(U2-Pad1) -> 3V3
- U2 pad 23: Net-(U2-Pad23) -> GND
- U2 pad 24: Net-(U2-Pad24) -> 3V3
- U2 pad 28: Net-(U2-Pad28) -> RGB_3V3
- U2 pad 34: Net-(U2-Pad34) -> SWDIO
- U2 pad 35: Net-(U2-Pad35) -> GND
- U2 pad 36: Net-(U2-Pad36) -> 3V3
- U2 pad 37: Net-(U2-Pad37) -> SWCLK
- U2 pad 44: Net-(U2-Pad44) -> BOOT0
- U2 pad 48: Net-(U2-Pad48) -> 3V3
- U2 pad 7: Net-(U2-Pad7) -> nRST
- U2 pad 8: Net-(U2-Pad8) -> GND
- U2 pad 9: Net-(U2-Pad9) -> 3V3
Routing:
- net Net-(Q1-Pad3): track 0.00 -> 1762.9 mm
- net 5V: track 17.4 -> 962.3 mm, vias 0 -> 18
- net Row4: track 0.00 -> 308.9 mm, vias 0 -> 1
- net Row2: track 0.00 -> 293.1 mm
- net Row1: track 0.00 -> 287.3 mm
- net Row3: track 0.00 -> 256.2 mm
- net RGB_3V3: track 0.00 -> 234.3 mm, vias 0 -> 2
- net nRST: track 0.00 -> 207.6 mm, vias 0 -> 2
- net Net-(U2-Pad31): track 0.00 -> 196.1 mm
- net SWDIO: track 0.00 -> 194.5 mm, vias 0 -> 1
- net Net-(J2-Pad1): track 0.00 -> 194.3 mm
- net SWCLK: track 0.00 -> 190.5 mm, vias 0 -> 1
- net Net-(U2-Pad30): track 0.00 -> 169.2 mm
- net Net-(U2-Pad29): track 0.00 -> 149.5 mm
- net Col13: track 0.00 -> 138.0 mm
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